File: ESP32_Motor/ESP32_Motor.kicad_pcb (KiCad board)
At the start: 2 copper layers, 78.5 x 60.5 mm, 18 parts, among them J1 Screw_Terminal_01x02, J2 Screw_Terminal_01x02, Q1 IRLML9301, Q2 BC847, U2 YD-ESP32-S3

Commit message: M_5_3_22_08_26
Parts:
- moved C2 35.2 mm to (123.3, 106.8)
- moved C3 34.9 mm to (123.4, 109.8)
- moved Q2 34.7 mm to (160.8, 85.2), turned to -90 degrees
- moved R5 34.6 mm to (160.8, 82.2), turned to 180 degrees
- moved R4 34.5 mm to (160.8, 79.8), turned to 0 degrees
- moved C1 34.3 mm to (116.9, 99.3)
- moved C4 34.3 mm to (123.4, 116.3)
- moved C5 34.3 mm to (126.7, 123.7)
- moved D1 34.3 mm to (121.4, 100.8)
- moved D2 34.3 mm to (164.2, 92.6)
- moved F1 34.3 mm to (121.2, 94.2)
- moved J1 34.3 mm to (106.8, 94.2)
- moved J2 34.3 mm to (172.8, 100.8)
- moved L1 34.3 mm to (124.4, 113.3)
- moved Q1 34.3 mm to (125.4, 100.3)
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Routing:
- net Net-(D2-A): track 39.2 -> 29.1 mm
- net +5VP: track 123.6 -> 118.6 mm
- net Net-(Q2-B): track 9.19 -> 4.65 mm
- net Net-(U2-GPIO1): track 5.34 -> 3.65 mm
Other:
- board size 78.5 x 60.5 mm -> 80.5 x 63.2 mm
- board text added: "+"
- board text added: "-"
- board text added: "Motor"

Commit message: M_5_5_26_08_26
Parts:
- added C6: 0.1u, Capacitor_SMD:C_0805_2012Metric, F.Cu at (116.6, 89.8)
- added R2: 4.7K, Resistor_SMD:R_0805_2012Metric_Pad1.20x1.40mm_HandSolder, F.Cu at (124.6, 89.9)
- added REF**: MountingHole_3.5mm, MountingHole:MountingHole_3.5mm, F.Cu at (142.5, 142.7)
- added REF**: MountingHole_3.5mm, MountingHole:MountingHole_3.5mm, F.Cu at (142.2, 51.3)
- added U1: DS18B20, Package_TO_SOT_THT:TO-92_Inline, F.Cu at (120.9, 91.4)
- D1: value BZT52B12V -> BZT52B5V6
- moved D1 5.33 mm to (121.2, 106.2)
- moved C1 5.23 mm to (116.8, 104.6)
- moved C2 5.23 mm to (123.2, 112.0)
- moved C3 5.23 mm to (123.3, 115.0)
- moved C4 5.23 mm to (123.3, 121.6)
- moved F1 5.23 mm to (121.1, 99.4)
- moved J1 5.23 mm to (106.7, 99.4)
- moved L1 5.23 mm to (124.3, 118.5)
- moved Q1 5.23 mm to (125.3, 105.6)
- moved R1 5.23 mm to (116.8, 108.1)
- moved D2 3.90 mm to (164.2, 96.5)
- moved J2 3.90 mm to (172.7, 104.6)
- moved RV1 2.92 mm to (118.6, 76.8)
- moved Q2 0.09 mm to (160.8, 85.3)
- moved R4 0.09 mm to (160.8, 79.8)
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Connections:
- net Net-(RV1-Pad3) renamed +3V3
- U2 pad 5: unconnected-(U2-GPIO5-Pad5) -> Net-(U1-DQ)
Routing:
- net +3V3: track 19.6 -> 45.0 mm
- net Net-(U1-DQ): track 0.00 -> 17.7 mm
- net +5VP: track 118.6 -> 111.1 mm
- net +5V: track 14.1 -> 9.08 mm
- net Net-(D2-A): track 29.1 -> 32.9 mm
- net Net-(U2-GPIO4): track 5.56 -> 7.50 mm
Other:
- board size 80.5 x 63.2 mm -> 105.9 x 105.9 mm

Commit message: M_5_5_27_08_26
Parts:
- removed REF** (x2): MountingHole_3.5mm, MountingHole:MountingHole_3.5mm
- added D3: FYLS-0805GD, LED_SMD:LED_0805_2012Metric, F.Cu at (167.5, 80.8)
- added Q3: PDTC143ZT, Package_TO_SOT_SMD:SOT-23, F.Cu at (162.7, 80.6)
- added R3: 1K, Resistor_SMD:R_0805_2012Metric_Pad1.20x1.40mm_HandSolder, F.Cu at (168.4, 84.3)
- moved Q2 6.25 mm to (160.8, 91.5)
- moved R4 6.25 mm to (160.7, 86.1)
- moved R5 6.25 mm to (160.8, 88.5)
Connections:
- R4 pad 1: Net-(U2-GPIO1) -> Net-(U2-GPIO2)
- U2 pad 40: unconnected-(U2-GPIO2-Pad40) -> Net-(U2-GPIO2)
- U2 pad 41: Net-(U2-GPIO1) -> Net-(Q3-B)
Routing:
- net +5VP: track 111.1 -> 124.1 mm
- net +3V3: track 45.0 -> 52.5 mm
- net Net-(U2-GPIO2): track 0.00 -> 7.21 mm
- net Net-(D2-A): track 32.9 -> 26.7 mm
- net Net-(Q3-B): track 0.00 -> 5.65 mm
- net Net-(U2-GPIO1): track 3.65 -> 0.00 mm
- net Net-(D3-K): track 0.00 -> 2.93 mm
- net Net-(D3-A): track 0.00 -> 2.93 mm
