File: ESP32_Motor/ESP32_Motor.kicad_sch (KiCad schematic)
At the start: 20 parts, among them J1 Conn_01x03, M1 Motor_DC, Q1 IRLML9301, Q2 Q_NPN_EBC, SW1 RotaryEncoder_Switch, U1 AMS1117-3.3, U2 YD-ESP32-S3

Commit message: M_5_2_19_08_26
Parts:
- removed C5: C, symbol Device:C
- removed J1: Conn_01x03, symbol Connector_Generic:Conn_01x03
- removed M1: Motor_DC, symbol Motor:Motor_DC
- removed Q2: Q_NPN_EBC, symbol Transistor_BJT:Q_NPN_EBC
- removed R2, R3: 4.7K, symbol Device:R_Small
- removed SW1: RotaryEncoder_Switch, symbol Device:RotaryEncoder_Switch
- removed U1: AMS1117-3.3, Package_TO_SOT_SMD:SOT-223-3_TabPin2, symbol Regulator_Linear:AMS1117-3.3
- added C5: 0.1u, Capacitor_SMD:C_0805_2012Metric, symbol Device:C_Small
- added F1: Polyfuse, Fuse:Fuse_Bourns_MF-SM_7.98x5.44mm, symbol Device:Polyfuse
- added J1, J2: Screw_Terminal_01x02, TerminalBlock_Phoenix:TerminalBlock_Phoenix_MKDS-1,5-2-5.08_1x02_P5.08mm_Horizontal, symbol Connector:Screw_Terminal_01x02
- added L1: L, Inductor_SMD:L_0805_2012Metric, symbol Device:L
- added Q2: BC847, Package_TO_SOT_SMD:SOT-23, symbol Transistor_BJT:BC847
- C1, C2, C3: footprint (none) -> Capacitor_SMD:C_0805_2012Metric
- C4: value C -> 0.1u; footprint (none) -> Capacitor_SMD:C_0805_2012Metric
- D1: value BZT52Bxx -> BZT52B12V
- R1: value R_Small -> 100K; footprint (none) -> Resistor_SMD:R_0805_2012Metric_Pad1.20x1.40mm_HandSolder
- R4: value 4.7K -> 1K; footprint (none) -> Resistor_SMD:R_0805_2012Metric_Pad1.20x1.40mm_HandSolder
- R5: value 4.7K -> 10K; footprint (none) -> Resistor_SMD:R_0805_2012Metric_Pad1.20x1.40mm_HandSolder
- RV1: value R_Potentiometer -> 10k; footprint (none) -> Potentiometer_SMD:Potentiometer_ACP_CA14-VSMD_Vertical
- U2: footprint Shared:YD-ESP32-S3 -> YD-ESP32-S3-main:YD-ESP32-S3
Connections:
- net GND: now also C5.2, J1.2 (Pin_2), Q2.2 (E)
- net at R4.2, R5.1: now also Q2.1 (B)
- net at D2.2 (A): now also J2.1 (Pin_1), Q2.3 (C)
- net +5VP: now reaches C2.1, C3.1, D1.1 (K), Q1.2 (S)
- net +5VP: now also D2.1 (K), J2.2 (Pin_2), L1.1
- net at U2.10 (GPIO17): no longer R4.1
- net +5V: now reaches U2.21 (5V)
- net +5V: now also C4.1, C5.1, L1.2
- net at U2.41 (GPIO1): now also R4.1
- net +3.3V: no longer names the net of RV1.3, U2.1 (3V3)
- net +3.3V: no longer C4.1
- net +5.0V: no longer names the net of Q1.3 (D)
- net +5.0V: now also F1.2; no longer D2.1 (K)
- new net: F1.1, J1.1 (Pin_1)
- no-connect marks 0 -> 37
Other:
- note added: "+Voud"
- note added: "-Vout"
- note added: "DC Motor"
- note added: "Vin+"
- note added: "Vin-"
- moved on the sheet: C1, C2, C3, C4, D1, D2, Q1, R1, R4, R5, RV1, U2

Commit message: M_5_3_22_08_26
Parts:
- D1: value BZT52B12V -> BZT52B5V6
Other:
- moved on the sheet: J1
Changed lines of the file:
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@@
 	(text "Vin-"
 		(exclude_from_sim no)
-		(at 36.576 62.484 0)
+		(at 41.656 62.484 0)
 		(effects
 			(font
@@
 	(text "Vin+"
 		(exclude_from_sim no)
-		(at 36.322 59.69 0)
+		(at 41.402 59.69 0)
 		(effects
 			(font
@@
 	)
 	(junction
-		(at 45.72 68.58)
+		(at 50.8 68.58)
 		(diameter 0)
 		(color 0 0 0 0)
@@
 	(wire
 		(pts
-			(xy 45.72 68.58) (xy 52.07 68.58)
+			(xy 50.8 68.58) (xy 57.15 68.58)
 		)
 		(stroke
@@
 	(wire
 		(pts
-			(xy 45.72 59.69) (xy 53.34 59.69)
-		)
-		(stroke
-			(width 0)
-			(type default)
-		)
-	)
-	(wire
-		(pts
 			(xy 171.45 107.95) (xy 175.26 107.95)
 		)
@@
 	(wire
 		(pts
-			(xy 45.72 68.58) (xy 45.72 69.85)
+			(xy 50.8 68.58) (xy 50.8 69.85)
 		)
 		(stroke
@@
 	(wire
 		(pts
-			(xy 45.72 62.23) (xy 45.72 68.58)
+			(xy 50.8 62.23) (xy 50.8 68.58)
 		)
 		(stroke
@@
 	(wire
 		(pts
+			(xy 50.8 59.69) (xy 53.34 59.69)
+		)
+		(stroke
+			(width 0)
+			(type default)
+		)
+	)
+	(wire
+		(pts
 			(xy 73.66 59.69) (xy 86.36 59.69)
 		)
@@
 			)
 		)
-		(property "Value" "BZT52B12V"
+		(property "Value" "BZT52B5V6"
 			(at 72.898 56.134 90)
 			(show_name no)
@@
 	(symbol
 		(lib_id "power:GND")
-		(at 45.72 69.85 0)
+		(at 50.8 69.85 0)
 		(unit 1)
 		(body_style 1)
@@
 		(fields_autoplaced yes)
 		(property "Reference" "#PWR04"
-			(at 45.72 76.2 0)
+			(at 50.8 76.2 0)
 			(hide yes)
 			(show_name no)
@@
 		)
 		(property "Value" "GND"
-			(at 45.72 74.93 0)
+			(at 50.8 74.93 0)
 			(show_name no)
 			(do_not_autoplace no)
@@
 		)
 		(property "Footprint" ""
-			(at 45.72 69.85 0)
+			(at 50.8 69.85 0)
 			(hide yes)
 			(show_name no)
@@
 		)
 		(property "Datasheet" ""
-			(at 45.72 69.85 0)
+			(at 50.8 69.85 0)
 			(hide yes)
 			(show_name no)
@@
 		)
 		(property "Description" "Power symbol creates a global label with name \"GND\" , ground"
-			(at 45.72 69.85 0)
+			(at 50.8 69.85 0)
 			(hide yes)
 			(show_name no)
@@
 	(symbol
 		(lib_id "power:PWR_FLAG")
-		(at 52.07 68.58 0)
+		(at 57.15 68.58 0)
 		(unit 1)
 		(body_style 1)
@@
 		(fields_autoplaced yes)
 		(property "Reference" "#FLG02"
-			(at 52.07 66.675 0)
+			(at 57.15 66.675 0)
 			(hide yes)
 			(show_name no)
@@
 		)
 		(property "Value" "PWR_FLAG"
-			(at 52.07 63.5 0)
+			(at 57.15 63.5 0)
 			(show_name no)
 			(do_not_autoplace no)
@@
 		)
 		(property "Footprint" ""
-			(at 52.07 68.58 0)
+			(at 57.15 68.58 0)
 			(hide yes)
 			(show_name no)
@@
 		)
 		(property "Datasheet" ""
-			(at 52.07 68.58 0)
+			(at 57.15 68.58 0)
 			(hide yes)
 			(show_name no)
@@
 		)
 		(property "Description" "Special symbol for telling ERC where power comes from"
-			(at 52.07 68.58 0)
+			(at 57.15 68.58 0)
 			(hide yes)
 			(show_name no)
@@
 	(symbol
 		(lib_id "Connector:Screw_Terminal_01x02")
-		(at 40.64 59.69 0)
+		(at 45.72 59.69 0)
 		(mirror y)
 		(unit 1)
@@
 		(dnp no)
 		(property "Reference" "J1"
-			(at 40.386 56.134 0)
+			(at 45.466 56.134 0)
 			(show_name no)
 			(do_not_autoplace no)
@@
 		)
 		(property "Value" "Screw_Terminal_01x02"
-			(at 39.116 68.326 0)
+			(at 44.196 68.326 0)
 			(hide yes)
 			(show_name no)
@@
 		)
 		(property "Footprint" "TerminalBlock_Phoenix:TerminalBlock_Phoenix_MKDS-1,5-2-5.08_1x02_P5.08mm_Horizontal"
-			(at 40.64 59.69 0)
+			(at 45.72 59.69 0)
 			(hide yes)
 			(show_name no)
@@
 		)
 		(property "Datasheet" ""
-			(at 40.64 59.69 0)
+			(at 45.72 59.69 0)
 			(hide yes)
 			(show_name no)
@@
 		)
 		(property "Description" "Generic screw terminal, single row, 01x02, script generated (kicad-library-utils/schlib/autogen/connector/)"
-			(at 40.64 59.69 0)
+			(at 45.72 59.69 0)
 			(hide yes)
 			(show_name no)

Commit message: M_5_5_26_08_26
Parts:
- added C6: 0.1u, Capacitor_SMD:C_0805_2012Metric, symbol Device:C
- added R2: 4.7K, Resistor_SMD:R_0805_2012Metric_Pad1.20x1.40mm_HandSolder, symbol Device:R_Small
- added U1: DS18B20, Package_TO_SOT_THT:TO-92_Inline, symbol Sensor_Temperature:DS18B20
Connections:
- net GND: now also C6.2, U1.1 (GND)
- net +3V3: now reaches RV1.3, U2.1 (3V3)
- net +3V3: now also C6.1, R2.1, U1.3 (V_{DD})
- net at U2.5 (GPIO5): now also R2.2, U1.2 (DQ)
- no-connect marks 37 -> 36
Other:
- moved on the sheet: RV1

Commit message: M_5_5_27_08_26
Parts:
- added D3: FYLS-0805GD, LED_SMD:LED_0805_2012Metric, symbol Device:LED_Small
- added Q3: PDTC143ZT, Package_TO_SOT_SMD:SOT-23, symbol Transistor_BJT:Q_NPN_BRT_BEC
- added R3: 1K, Resistor_SMD:R_0805_2012Metric_Pad1.20x1.40mm_HandSolder, symbol Device:R_Small
Connections:
- net +5VP: now also R3.1
- net GND: now also Q3.2 (E)
- net at U2.40 (GPIO2): now also R4.1
- net at U2.41 (GPIO1): now also Q3.1 (B); no longer R4.1
- new net: D3.1 (K), Q3.3 (C)
- new net: D3.2 (A), R3.2
- no-connect marks 36 -> 35
Other:
- moved on the sheet: C5, D2, J2, Q2, R4, R5
